File: hardware/ec60-nrf52840/analog.kicad_sch (KiCad schematic)
At the start: 25 parts, among them U2 74HC4051, U3 OPA350, U4 74HC4051

Commit message: fix: validate single-nRF PCB and add 3D renders
Complete routing and native clearance repairs, freeze footprint metadata, and preserve EC60 sensing and mounting geometry. Add reproducible KiCad stills and a six-second 3D turntable with model provenance.

Validation: strict DRC 0 errors and 0 opens; ERC 0 errors; 268 physical pin pairs pass with no connectivity regressions. Render source hashes are unchanged, and MP4/GIF decoding passes. Physical assembly and SI/RF validation remain pending.
Parts:
- C10: footprint Capacitor_SMD:C_0402_1005Metric -> YAECKB:C_0402_1005Metric__C10
- C11: footprint Capacitor_SMD:C_0402_1005Metric -> YAECKB:C_0402_1005Metric__C11
- C12: footprint Capacitor_SMD:C_0402_1005Metric -> YAECKB:C_0402_1005Metric__C12
- C9: footprint Capacitor_SMD:C_0402_1005Metric -> YAECKB:C_0402_1005Metric__C9
- JP1: footprint Resistor_SMD:R_0603_1608Metric_Pad0.98x0.95mm_HandSolder -> YAECKB:R_0603_1608Metric_Pad0.98x0.95mm_HandSolder__JP1
- R10: footprint Resistor_SMD:R_0402_1005Metric -> YAECKB:R_0402_1005Metric__R10
- R11: footprint Resistor_SMD:R_0402_1005Metric -> YAECKB:R_0402_1005Metric__R11
- R12: footprint Resistor_SMD:R_0402_1005Metric -> YAECKB:R_0402_1005Metric__R12
- R13: footprint Resistor_SMD:R_0402_1005Metric -> YAECKB:R_0402_1005Metric__R13
- R14: footprint Resistor_SMD:R_0402_1005Metric -> YAECKB:R_0402_1005Metric__R14
- R15: footprint Resistor_SMD:R_0402_1005Metric -> YAECKB:R_0402_1005Metric__R15
- R16: footprint Resistor_SMD:R_0402_1005Metric -> YAECKB:R_0402_1005Metric__R16
- R17: footprint Resistor_SMD:R_0402_1005Metric -> YAECKB:R_0402_1005Metric__R17
- R18: footprint Resistor_SMD:R_0402_1005Metric -> YAECKB:R_0402_1005Metric__R18
- R19: footprint Resistor_SMD:R_0402_1005Metric -> YAECKB:R_0402_1005Metric__R19
- R20: footprint Resistor_SMD:R_0402_1005Metric -> YAECKB:R_0402_1005Metric__R20
- R21: footprint Resistor_SMD:R_0402_1005Metric -> YAECKB:R_0402_1005Metric__R21
- R23: footprint Resistor_SMD:R_0402_1005Metric -> YAECKB:R_0402_1005Metric__R23
- R24: footprint Resistor_SMD:R_0402_1005Metric -> YAECKB:R_0402_1005Metric__R24
- R25: footprint Resistor_SMD:R_0402_1005Metric -> YAECKB:R_0402_1005Metric__R25
- R8: footprint Resistor_SMD:R_0402_1005Metric -> YAECKB:R_0402_1005Metric__R8
- R9: footprint Resistor_SMD:R_0402_1005Metric -> YAECKB:R_0402_1005Metric__R9
- U2: footprint YAECKB:TSSOP16 -> YAECKB:TSSOP16__U2
- U3: footprint Package_SO:SOIC-8_3.9x4.9mm_P1.27mm -> YAECKB:SOIC-8_3.9x4.9mm_P1.27mm__U3
- U4: footprint YAECKB:TSSOP16 -> YAECKB:TSSOP16__U4
