File: hardware/ec60-nrf52840/matrix.kicad_sch (KiCad schematic)
At the start: 74 parts, among them SW10 EC_SW, SW11 EC_SW, SW12 EC_SW, SW13 EC_SW, SW14 EC_SW, SW15 EC_SW, SW16 EC_SW, SW17 EC_SW, SW18 EC_SW, SW19 EC_SW, SW2 EC_SW, SW20 EC_SW, SW21 EC_SW, SW22 EC_SW, SW23 EC_SW, SW24 EC_SW, SW25 EC_SW, SW26 EC_SW, SW27 EC_SW, SW28 EC_SW, SW29 EC_SW, SW3 EC_SW, SW30 EC_SW, SW31 ANSI_\, SW32 ISO_Enter, SW33 EC_SW, SW34 EC_SW, SW35 EC_SW, SW36 EC_SW, SW37 EC_SW, SW38 EC_SW, SW39 EC_SW, SW4 EC_SW, SW40 EC_SW, SW41 EC_SW, SW42 EC_SW, SW43 EC_SW, SW44 EC_SW, SW45 ISO_|, SW46 ANSI_Enter, SW47 EC_SW, SW48 EC_SW, SW49 EC_SW, SW5 EC_SW, SW50 EC_SW, SW51 EC_SW, SW52 EC_SW, SW53 EC_SW, SW54 EC_SW, SW55 EC_SW, SW56 EC_SW, SW57 EC_SW, SW58 EC_SW, SW59 EC_SW, SW6 EC_SW, SW60 EC_SW_1u&1.75u, SW61 EC_SW, SW62 EC_SW_1u&1.75u, SW63 EC_SW, SW64 EC_SW, SW65 EC_SW, SW66 EC_SW, SW67 EC_SW, SW68 EC_SW, SW69 EC_SW, SW7 EC_SW, SW70 EC_SW, SW71 EC_SW, SW72 EC_SW, SW73 EC_SW, SW74 EC_SW, SW75 EC_SW, SW8 EC_SW, SW9 EC_SW

Commit message: fix: validate single-nRF PCB and add 3D renders
Complete routing and native clearance repairs, freeze footprint metadata, and preserve EC60 sensing and mounting geometry. Add reproducible KiCad stills and a six-second 3D turntable with model provenance.

Validation: strict DRC 0 errors and 0 opens; ERC 0 errors; 268 physical pin pairs pass with no connectivity regressions. Render source hashes are unchanged, and MP4/GIF decoding passes. Physical assembly and SI/RF validation remain pending.
Parts:
- SW10: footprint YAECKB:ecs_pad_no_ring -> YAECKB:ecs_pad_no_ring__SW10; now left out of the parts list
- SW11: footprint YAECKB:ecs_pad_no_ring -> YAECKB:ecs_pad_no_ring__SW11; now left out of the parts list
- SW12: footprint YAECKB:ecs_pad_no_ring -> YAECKB:ecs_pad_no_ring__SW12; now left out of the parts list
- SW13: footprint YAECKB:ecs_pad_no_ring -> YAECKB:ecs_pad_no_ring__SW13; now left out of the parts list
- SW14: footprint YAECKB:ecs_pad_no_ring -> YAECKB:ecs_pad_no_ring__SW14; now left out of the parts list
- SW15: footprint YAECKB:ecs_pad_no_ring -> YAECKB:ecs_pad_no_ring__SW15; now left out of the parts list
- SW16: footprint YAECKB:ecs_pad_no_ring -> YAECKB:ecs_pad_no_ring__SW16; now left out of the parts list
- SW17: footprint YAECKB:ecs_pad_no_ring -> YAECKB:ecs_pad_no_ring__SW17; now left out of the parts list
- SW18: footprint YAECKB:ecs_pad_no_ring -> YAECKB:ecs_pad_no_ring__SW18; now left out of the parts list
- SW19: footprint YAECKB:ecs_pad_no_ring -> YAECKB:ecs_pad_no_ring__SW19; now left out of the parts list
- SW2: footprint YAECKB:ecs_pad_no_ring -> YAECKB:ecs_pad_no_ring__SW2; now left out of the parts list
- SW20: footprint YAECKB:ecs_pad_no_ring -> YAECKB:ecs_pad_no_ring__SW20; now left out of the parts list
- SW21: footprint YAECKB:ecs_pad_no_ring -> YAECKB:ecs_pad_no_ring__SW21; now left out of the parts list
- SW22: footprint YAECKB:ecs_pad_no_ring -> YAECKB:ecs_pad_no_ring__SW22; now left out of the parts list
- SW23: footprint YAECKB:ecs_pad_no_ring -> YAECKB:ecs_pad_no_ring__SW23; now left out of the parts list
- SW24: footprint YAECKB:ecs_pad_no_ring -> YAECKB:ecs_pad_no_ring__SW24; now left out of the parts list
- SW25: footprint YAECKB:ecs_pad_no_ring -> YAECKB:ecs_pad_no_ring__SW25; now left out of the parts list
- SW26: footprint YAECKB:ecs_pad_no_ring -> YAECKB:ecs_pad_no_ring__SW26; now left out of the parts list
- SW27: footprint YAECKB:ecs_pad_no_ring -> YAECKB:ecs_pad_no_ring__SW27; now left out of the parts list
- SW28: footprint YAECKB:ecs_pad_no_ring -> YAECKB:ecs_pad_no_ring__SW28; now left out of the parts list
- SW29: footprint YAECKB:ecs_pad_no_ring -> YAECKB:ecs_pad_no_ring__SW29; now left out of the parts list
- SW3: footprint YAECKB:ecs_pad_no_ring -> YAECKB:ecs_pad_no_ring__SW3; now left out of the parts list
- SW30: footprint YAECKB:ecs_pad_no_ring -> YAECKB:ecs_pad_no_ring__SW30; now left out of the parts list
- SW31: footprint YAECKB:ecs_pad_no_ring -> YAECKB:ecs_pad_no_ring__SW31; now left out of the parts list
- SW32: footprint YAECKB:ecs_pad_no_ring -> YAECKB:ecs_pad_no_ring__SW32; now left out of the parts list
- SW33: footprint YAECKB:ecs_pad_no_ring_stepped&normal -> YAECKB:ecs_pad_no_ring_stepped&normal__SW33; now left out of the parts list
- SW34: footprint YAECKB:ecs_pad_no_ring -> YAECKB:ecs_pad_no_ring__SW34; now left out of the parts list
- SW35: footprint YAECKB:ecs_pad_no_ring -> YAECKB:ecs_pad_no_ring__SW35; now left out of the parts list
- SW36: footprint YAECKB:ecs_pad_no_ring -> YAECKB:ecs_pad_no_ring__SW36; now left out of the parts list
- SW37: footprint YAECKB:ecs_pad_no_ring -> YAECKB:ecs_pad_no_ring__SW37; now left out of the parts list
- SW38: footprint YAECKB:ecs_pad_no_ring -> YAECKB:ecs_pad_no_ring__SW38; now left out of the parts list
- SW39: footprint YAECKB:ecs_pad_no_ring -> YAECKB:ecs_pad_no_ring__SW39; now left out of the parts list
- SW4: footprint YAECKB:ecs_pad_no_ring -> YAECKB:ecs_pad_no_ring__SW4; now left out of the parts list
- SW40: footprint YAECKB:ecs_pad_no_ring -> YAECKB:ecs_pad_no_ring__SW40; now left out of the parts list
- SW41: footprint YAECKB:ecs_pad_no_ring -> YAECKB:ecs_pad_no_ring__SW41; now left out of the parts list
- SW42: footprint YAECKB:ecs_pad_no_ring -> YAECKB:ecs_pad_no_ring__SW42; now left out of the parts list
- SW43: footprint YAECKB:ecs_pad_no_ring -> YAECKB:ecs_pad_no_ring__SW43; now left out of the parts list
- SW44: footprint YAECKB:ecs_pad_no_ring -> YAECKB:ecs_pad_no_ring__SW44; now left out of the parts list
- SW45: footprint YAECKB:ecs_pad_no_ring -> YAECKB:ecs_pad_no_ring__SW45; now left out of the parts list
- SW46: footprint YAECKB:ecs_pad_no_ring -> YAECKB:ecs_pad_no_ring__SW46; now left out of the parts list
- SW47: footprint YAECKB:ecs_pad_no_ring -> YAECKB:ecs_pad_no_ring__SW47; now left out of the parts list
- SW48: footprint YAECKB:ecs_pad_no_ring_1u_edge_cut -> YAECKB:ecs_pad_no_ring_1u_edge_cut__SW48; now left out of the parts list
- SW49: footprint YAECKB:ecs_pad_no_ring_1u_edge_cut -> YAECKB:ecs_pad_no_ring_1u_edge_cut__SW49; now left out of the parts list
- SW5: footprint YAECKB:ecs_pad_no_ring -> YAECKB:ecs_pad_no_ring__SW5; now left out of the parts list
- SW50: footprint YAECKB:ecs_pad_no_ring -> YAECKB:ecs_pad_no_ring__SW50; now left out of the parts list
- SW51: footprint YAECKB:ecs_pad_no_ring -> YAECKB:ecs_pad_no_ring__SW51; now left out of the parts list
- SW52: footprint YAECKB:ecs_pad_no_ring -> YAECKB:ecs_pad_no_ring__SW52; now left out of the parts list
- SW53: footprint YAECKB:ecs_pad_no_ring -> YAECKB:ecs_pad_no_ring__SW53; now left out of the parts list
- SW54: footprint YAECKB:ecs_pad_no_ring -> YAECKB:ecs_pad_no_ring__SW54; now left out of the parts list
- SW55: footprint YAECKB:ecs_pad_no_ring -> YAECKB:ecs_pad_no_ring__SW55; now left out of the parts list
- SW56: footprint YAECKB:ecs_pad_no_ring -> YAECKB:ecs_pad_no_ring__SW56; now left out of the parts list
- SW57: footprint YAECKB:ecs_pad_no_ring -> YAECKB:ecs_pad_no_ring__SW57; now left out of the parts list
- SW58: footprint YAECKB:ecs_pad_no_ring -> YAECKB:ecs_pad_no_ring__SW58; now left out of the parts list
- SW59: footprint YAECKB:ecs_pad_no_ring -> YAECKB:ecs_pad_no_ring__SW59; now left out of the parts list
- SW6: footprint YAECKB:ecs_pad_no_ring -> YAECKB:ecs_pad_no_ring__SW6; now left out of the parts list
- SW60: footprint YAECKB:ecs_pad_no_ring_1u1.75u -> YAECKB:ecs_pad_no_ring_1u1.75u__SW60; now left out of the parts list
- SW61: footprint YAECKB:ecs_pad_no_ring -> YAECKB:ecs_pad_no_ring__SW61; now left out of the parts list
- SW62: footprint YAECKB:ecs_pad_no_ring_1u1.75u -> YAECKB:ecs_pad_no_ring_1u1.75u__SW62; now left out of the parts list
- SW63: footprint YAECKB:ecs_pad_no_ring -> YAECKB:ecs_pad_no_ring__SW63; now left out of the parts list
- SW64: footprint YAECKB:ecs_pad_no_ring -> YAECKB:ecs_pad_no_ring__SW64; now left out of the parts list
- SW65: footprint YAECKB:ecs_pad_no_ring -> YAECKB:ecs_pad_no_ring__SW65; now left out of the parts list
- SW66: footprint YAECKB:ecs_pad_no_ring -> YAECKB:ecs_pad_no_ring__SW66; now left out of the parts list
- SW67: footprint YAECKB:ecs_pad_no_ring -> YAECKB:ecs_pad_no_ring__SW67; now left out of the parts list
- SW68: footprint YAECKB:ecs_pad_no_ring_stepped&normal -> YAECKB:ecs_pad_no_ring_stepped&normal__SW68; now left out of the parts list
- SW69: footprint YAECKB:ecs_pad_no_ring_stepped&normal -> YAECKB:ecs_pad_no_ring_stepped&normal__SW69; now left out of the parts list
- SW7: footprint YAECKB:ecs_pad_no_ring -> YAECKB:ecs_pad_no_ring__SW7; now left out of the parts list
- SW70: footprint YAECKB:ecs_pad_no_ring -> YAECKB:ecs_pad_no_ring__SW70; now left out of the parts list
- SW71: footprint YAECKB:ecs_pad_no_ring_stepped&normal -> YAECKB:ecs_pad_no_ring_stepped&normal__SW71; now left out of the parts list
- SW72: footprint YAECKB:ecs_pad_no_ring -> YAECKB:ecs_pad_no_ring__SW72; now left out of the parts list
- SW73: footprint YAECKB:ecs_pad_no_ring -> YAECKB:ecs_pad_no_ring__SW73; now left out of the parts list
- SW74: footprint YAECKB:ecs_pad_no_ring -> YAECKB:ecs_pad_no_ring__SW74; now left out of the parts list
- SW75: footprint YAECKB:ecs_pad_no_ring -> YAECKB:ecs_pad_no_ring__SW75; now left out of the parts list
- SW8: footprint YAECKB:ecs_pad_no_ring -> YAECKB:ecs_pad_no_ring__SW8; now left out of the parts list
- SW9: footprint YAECKB:ecs_pad_no_ring -> YAECKB:ecs_pad_no_ring__SW9; now left out of the parts list
