File: hardware/ec60-nrf52840/mounting.kicad_sch (KiCad schematic)
At the start: 26 parts

Commit message: fix: validate single-nRF PCB and add 3D renders
Complete routing and native clearance repairs, freeze footprint metadata, and preserve EC60 sensing and mounting geometry. Add reproducible KiCad stills and a six-second 3D turntable with model provenance.

Validation: strict DRC 0 errors and 0 opens; ERC 0 errors; 268 physical pin pairs pass with no connectivity regressions. Render source hashes are unchanged, and MP4/GIF decoding passes. Physical assembly and SI/RF validation remain pending.
Parts:
- H1: footprint YAECKB:HOLE_M2 -> YAECKB:HOLE_M2__H1; now left out of the parts list
- H10: footprint YAECKB:HOLE_M2 -> YAECKB:HOLE_M2__H10; now left out of the parts list
- H11: footprint YAECKB:HOLE_M2 -> YAECKB:HOLE_M2__H11; now left out of the parts list
- H12: footprint YAECKB:HOLE_M2 -> YAECKB:HOLE_M2__H12; now left out of the parts list
- H13: footprint YAECKB:HOLE_M2 -> YAECKB:HOLE_M2__H13; now left out of the parts list
- H14: footprint YAECKB:HOLE_M2 -> YAECKB:HOLE_M2__H14; now left out of the parts list
- H15: footprint YAECKB:HOLE_M2 -> YAECKB:HOLE_M2__H15; now left out of the parts list
- H16: footprint YAECKB:HOLE_M2 -> YAECKB:HOLE_M2__H16; now left out of the parts list
- H17: footprint YAECKB:HOLE_M2 -> YAECKB:HOLE_M2__H17; now left out of the parts list
- H18: footprint YAECKB:HOLE_M2 -> YAECKB:HOLE_M2__H18; now left out of the parts list
- H19: footprint YAECKB:HOLE_M2 -> YAECKB:HOLE_M2__H19; now left out of the parts list
- H2: footprint YAECKB:HOLE_M2 -> YAECKB:HOLE_M2__H2; now left out of the parts list
- H20: footprint YAECKB:HOLE_M2 -> YAECKB:HOLE_M2__H20; now left out of the parts list
- H21: footprint YAECKB:HOLE_M2 -> YAECKB:HOLE_M2__H21; now left out of the parts list
- H22: footprint YAECKB:HOLE_M2 -> YAECKB:HOLE_M2__H22; now left out of the parts list
- H23: footprint YAECKB:HOLE_M2 -> YAECKB:HOLE_M2__H23; now left out of the parts list
- H24: footprint YAECKB:HOLE_M2 -> YAECKB:HOLE_M2__H24; now left out of the parts list
- H25: footprint YAECKB:HOLE_M2 -> YAECKB:HOLE_M2__H25; now left out of the parts list
- H26: footprint YAECKB:HOLE_M2 -> YAECKB:HOLE_M2__H26; now left out of the parts list
- H3: footprint YAECKB:HOLE_M2 -> YAECKB:HOLE_M2__H3; now left out of the parts list
- H4: footprint YAECKB:HOLE_M2 -> YAECKB:HOLE_M2__H4; now left out of the parts list
- H5: footprint YAECKB:HOLE_M2 -> YAECKB:HOLE_M2__H5; now left out of the parts list
- H6: footprint YAECKB:HOLE_M2 -> YAECKB:HOLE_M2__H6; now left out of the parts list
- H7: footprint YAECKB:HOLE_M2 -> YAECKB:HOLE_M2__H7; now left out of the parts list
- H8: footprint YAECKB:HOLE_M2 -> YAECKB:HOLE_M2__H8; now left out of the parts list
- H9: footprint YAECKB:HOLE_M2 -> YAECKB:HOLE_M2__H9; now left out of the parts list
