File: hardware/ec60-nrf52840/EC60-nRF52840.kicad_pcb (KiCad board)
At the start: 4 copper layers, 285 x 94.6 mm, 177 parts, among them J1 REAR_USB_DAUGHTERBOARD, J2 PROTECTED_1S_4V2_NTC10K, J3 SWD_POGO, SW1 EVQPUC02K_RESET, SW10 EC_SW, SW100 JS102011SAQN_POWER, SW11 EC_SW, SW12 EC_SW, SW13 EC_SW, SW14 EC_SW, SW15 EC_SW, SW16 EC_SW, SW17 EC_SW, SW18 EC_SW, SW19 EC_SW, SW2 EC_SW, SW20 EC_SW, SW21 EC_SW, SW22 EC_SW, SW23 EC_SW, SW24 EC_SW, SW25 EC_SW, SW26 EC_SW, SW27 EC_SW, SW28 EC_SW, SW29 EC_SW, SW3 EC_SW, SW30 EC_SW, SW31 ANSI_\, SW32 ISO_Enter, SW33 EC_SW, SW34 EC_SW, SW35 EC_SW, SW36 EC_SW, SW37 EC_SW, SW38 EC_SW, SW39 EC_SW, SW4 EC_SW, SW40 EC_SW, SW41 EC_SW, SW42 EC_SW, SW43 EC_SW, SW44 EC_SW, SW45 ISO_|, SW46 ANSI_Enter, SW47 EC_SW, SW48 EC_SW, SW49 EC_SW, SW5 EC_SW, SW50 EC_SW, SW51 EC_SW, SW52 EC_SW, SW53 EC_SW, SW54 EC_SW, SW55 EC_SW, SW56 EC_SW, SW57 EC_SW, SW58 EC_SW, SW59 EC_SW, SW6 EC_SW, SW60 EC_SW_1u&1.75u, SW61 EC_SW, SW62 EC_SW_1u&1.75u, SW63 EC_SW, SW64 EC_SW, SW65 EC_SW, SW66 EC_SW, SW67 EC_SW, SW68 EC_SW, SW69 EC_SW, SW7 EC_SW, SW70 EC_SW, SW71 EC_SW, SW72 EC_SW, SW73 EC_SW, SW74 EC_SW, SW75 EC_SW, SW8 EC_SW, SW9 EC_SW, U1 MDBT50Q-1MV2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

Commit message: feat: checkpoint HDI power layout and buildable YETI60 firmware
Routing:
- net BAT_CELL: track 71.1 -> 82.8 mm, vias 3 -> 5
- net +3.3V: track 316.1 -> 325.0 mm, vias 6 -> 9
- net USB_5V: track 301.1 -> 307.3 mm, vias 9 -> 11

Commit message: docs: add YETI60 procurement BOM and remove decorative board branding
Other:
- board text removed: "YETI60 / EC60 by Cipulot"
Changed lines of the file:
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@@
 		(layer "B.Fab")
-	)
-	(gr_text "YETI60 / EC60 by Cipulot"
-		(at 214 141.5 0)
-		(layer "B.SilkS")
-		(effects
-			(font
-				(size 0.8 0.8)
-				(thickness 0.12)
-			)
-			(justify mirror)
-		)
 	)
 	(gr_text "NRF-1.0-dev / REAR USB"
