File: hardware/ec60-nrf52840/EC60-nRF52840.kicad_pcb (KiCad board)
At the start: 4 copper layers, 285 x 94.6 mm, 177 parts, among them J1 REAR_USB_DAUGHTERBOARD, J2 PROTECTED_1S_4V2_NTC10K, J3 SWD_POGO, SW1 EVQPUC02K_RESET, SW10 EC_SW, SW100 JS102011SAQN_POWER, SW11 EC_SW, SW12 EC_SW, SW13 EC_SW, SW14 EC_SW, SW15 EC_SW, SW16 EC_SW, SW17 EC_SW, SW18 EC_SW, SW19 EC_SW, SW2 EC_SW, SW20 EC_SW, SW21 EC_SW, SW22 EC_SW, SW23 EC_SW, SW24 EC_SW, SW25 EC_SW, SW26 EC_SW, SW27 EC_SW, SW28 EC_SW, SW29 EC_SW, SW3 EC_SW, SW30 EC_SW, SW31 ANSI_\, SW32 ISO_Enter, SW33 EC_SW, SW34 EC_SW, SW35 EC_SW, SW36 EC_SW, SW37 EC_SW, SW38 EC_SW, SW39 EC_SW, SW4 EC_SW, SW40 EC_SW, SW41 EC_SW, SW42 EC_SW, SW43 EC_SW, SW44 EC_SW, SW45 ISO_|, SW46 ANSI_Enter, SW47 EC_SW, SW48 EC_SW, SW49 EC_SW, SW5 EC_SW, SW50 EC_SW, SW51 EC_SW, SW52 EC_SW, SW53 EC_SW, SW54 EC_SW, SW55 EC_SW, SW56 EC_SW, SW57 EC_SW, SW58 EC_SW, SW59 EC_SW, SW6 EC_SW, SW60 EC_SW_1u&1.75u, SW61 EC_SW, SW62 EC_SW_1u&1.75u, SW63 EC_SW, SW64 EC_SW, SW65 EC_SW, SW66 EC_SW, SW67 EC_SW, SW68 EC_SW, SW69 EC_SW, SW7 EC_SW, SW70 EC_SW, SW71 EC_SW, SW72 EC_SW, SW73 EC_SW, SW74 EC_SW, SW75 EC_SW, SW8 EC_SW, SW9 EC_SW, U1 MDBT50Q-1MV2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

Commit message: feat: make the 1600mAh single-cell pack the YETI60 default
Retain the C5 JSH daughterboard, revise BQ24074 charge programming and USB500 firmware, and synchronize the recessed case, bilingual engineering evidence and current renders. All 31 audit stages pass; supplier pack qualification and physical acceptance remain pending.
Parts:
- added R55: 69.8k/1%, YAECKB:R_0402_1005Metric__R55, B.Cu at (117.7, 148.4)
- added R56: 1.82k/1%, YAECKB:R_0402_1005Metric__R56, B.Cu at (115.1, 146.8)
- R40: value 8.87k/1% -> 2.21k/1%
- moved R40 0.55 mm to (116.7, 148.1)
Connections:
- U5 pad 14: unconnected-(U5-TMR-Pad14) -> TMR_SET
- U5 pad 15: unconnected-(U5-ITERM-Pad15) -> ITERM_SET
Routing:
- net ITERM_SET: track 0.00 -> 7.15 mm, vias 0 -> 2
- net USB_5V: track 307.3 -> 311.9 mm, vias 11 -> 10
- net GND: track 1707.2 -> 1709.6 mm
- net TMR_SET: track 0.00 -> 1.74 mm
- net ICHG_SET: track 0.40 -> 0.94 mm

Commit message: feat: support ordinary JLC fabrication and document complete materials
Parts:
- R56: value 1.82k/1% -> 1.69k/1%
- moved C40 6.22 mm to (123.5, 148.1)
- moved R56 2.90 mm to (117.7, 148.1)
- moved C41 1.55 mm to (119.6, 151.0)
- moved R55 1.01 mm to (118.7, 148.2)
Routing:
- net USB_5V: track 311.9 -> 299.3 mm, vias 10 -> 8
- net SWDIO: track 29.1 -> 41.3 mm, vias 2 -> 3
- net GND: track 1709.6 -> 1721.7 mm
- net BAT_CELL: track 82.8 -> 72.7 mm, vias 5 -> 3
- net +3.3V: track 325.0 -> 318.2 mm, vias 9 -> 6
- net ITERM_SET: track 7.15 -> 1.23 mm, vias 2 -> 0
- net ROW_DRV2: track 265.2 -> 269.2 mm
