File: hardware/ec60-nrf52840/power.kicad_sch (KiCad schematic)
At the start: 31 parts, among them J2 PROTECTED_1S_4V2_NTC10K, SW100 JS102011SAQN_POWER, U5 BQ24074RGT, U6 TPS63031DSK, U7 TPS22919DCK, U8 TPS22919DCK

Commit message: fix: validate single-nRF PCB and add 3D renders
Complete routing and native clearance repairs, freeze footprint metadata, and preserve EC60 sensing and mounting geometry. Add reproducible KiCad stills and a six-second 3D turntable with model provenance.

Validation: strict DRC 0 errors and 0 opens; ERC 0 errors; 268 physical pin pairs pass with no connectivity regressions. Render source hashes are unchanged, and MP4/GIF decoding passes. Physical assembly and SI/RF validation remain pending.
Parts:
- C40: footprint Capacitor_SMD:C_0603_1608Metric -> YAECKB:C_0603_1608Metric__C40
- C41: footprint Capacitor_SMD:C_0603_1608Metric -> YAECKB:C_0603_1608Metric__C41
- C42: footprint Capacitor_SMD:C_0603_1608Metric -> YAECKB:C_0603_1608Metric__C42
- C43: footprint Capacitor_SMD:C_0603_1608Metric -> YAECKB:C_0603_1608Metric__C43
- C44: footprint Capacitor_SMD:C_0603_1608Metric -> YAECKB:C_0603_1608Metric__C44
- C45: footprint Capacitor_SMD:C_0603_1608Metric -> YAECKB:C_0603_1608Metric__C45
- C46: footprint Capacitor_SMD:C_0603_1608Metric -> YAECKB:C_0603_1608Metric__C46
- C47: footprint Capacitor_SMD:C_0402_1005Metric -> YAECKB:C_0402_1005Metric__C47
- C48: footprint Capacitor_SMD:C_0402_1005Metric -> YAECKB:C_0402_1005Metric__C48
- J2: footprint Connector_JST:JST_PH_S3B-PH-SM4-TB_1x03-1MP_P2.00mm_Horizontal -> YAECKB:JST_PH_S3B-PH-SM4-TB_1x03-1MP_P2.00mm_Horizontal__J2
- L1: footprint Inductor_SMD:L_Wuerth_MAPI-3015 -> YAECKB:L_Wuerth_MAPI-3015__L1
- R40: footprint Resistor_SMD:R_0402_1005Metric -> YAECKB:R_0402_1005Metric__R40
- R41: footprint Resistor_SMD:R_0402_1005Metric -> YAECKB:R_0402_1005Metric__R41
- R42: footprint Resistor_SMD:R_0402_1005Metric -> YAECKB:R_0402_1005Metric__R42
- R43: footprint Resistor_SMD:R_0402_1005Metric -> YAECKB:R_0402_1005Metric__R43
- R44: footprint Resistor_SMD:R_0402_1005Metric -> YAECKB:R_0402_1005Metric__R44
- R45: footprint Resistor_SMD:R_0402_1005Metric -> YAECKB:R_0402_1005Metric__R45
- R46: footprint Resistor_SMD:R_0402_1005Metric -> YAECKB:R_0402_1005Metric__R46
- R47: footprint Resistor_SMD:R_0402_1005Metric -> YAECKB:R_0402_1005Metric__R47
- R48: footprint Resistor_SMD:R_0402_1005Metric -> YAECKB:R_0402_1005Metric__R48
- R49: footprint Resistor_SMD:R_0402_1005Metric -> YAECKB:R_0402_1005Metric__R49
- R50: footprint Resistor_SMD:R_0402_1005Metric -> YAECKB:R_0402_1005Metric__R50
- R51: footprint Resistor_SMD:R_0402_1005Metric -> YAECKB:R_0402_1005Metric__R51
- R52: footprint Resistor_SMD:R_0402_1005Metric -> YAECKB:R_0402_1005Metric__R52
- R53: footprint Resistor_SMD:R_0402_1005Metric -> YAECKB:R_0402_1005Metric__R53
- R54: footprint Resistor_SMD:R_0402_1005Metric -> YAECKB:R_0402_1005Metric__R54
- SW100: footprint Button_Switch_SMD:SW_SPDT_CK_JS102011SAQN -> YAECKB:SW_SPDT_CK_JS102011SAQN__SW100
- U5: footprint Package_DFN_QFN:VQFN-16-1EP_3x3mm_P0.5mm_EP1.6x1.6mm -> YAECKB:VQFN-16-1EP_3x3mm_P0.5mm_EP1.6x1.6mm__U5
- U6: footprint Package_SON:WSON-10-1EP_2.5x2.5mm_P0.5mm_EP1.2x2mm -> YAECKB:WSON-10-1EP_2.5x2.5mm_P0.5mm_EP1.2x2mm__U6
- U7: footprint Package_TO_SOT_SMD:SOT-363_SC-70-6 -> YAECKB:SOT-363_SC-70-6__U7
- U8: footprint Package_TO_SOT_SMD:SOT-363_SC-70-6 -> YAECKB:SOT-363_SC-70-6__U8

Commit message: feat: make the 1600mAh single-cell pack the YETI60 default
Retain the C5 JSH daughterboard, revise BQ24074 charge programming and USB500 firmware, and synchronize the recessed case, bilingual engineering evidence and current renders. All 31 audit stages pass; supplier pack qualification and physical acceptance remain pending.
Parts:
- added R55: 69.8k/1%, YAECKB:R_0402_1005Metric__R55, symbol YAECKB:R
- added R56: 1.82k/1%, YAECKB:R_0402_1005Metric__R56, symbol YAECKB:R
- R40: value 8.87k/1% -> 2.21k/1%
Connections:
- net GND: now also R55.2, R56.2
- net TMR_SET: now reaches U5.14 (TMR)
- net TMR_SET: now also R55.1
- net ITERM_SET: now reaches U5.15 (ITERM)
- net ITERM_SET: now also R56.1
- no-connect marks 4 -> 2
Other:
- note added: "P2: protected 1600mAh 1S 4.2V pack, third-wire 10k NTC; independent pack thermal interruption within actual cell 15..43C required"
- note added: "R40=2.21k: 403mA nominal; R55/TMR=69.8k, R56/ITERM=1.82k (all 1%). USB500 only after host configuration; suspend disables charging"
- note removed: "Default USB100; firmware controls EN1/EN2 for enumeration/suspend. ICHG approx 100mA. TMR/ITERM NC = datasheet defaults"
- note removed: "Protected 1S 4.2V Li-ion pack with 10k 103AT-2-compatible NTC required; J2 is not an unprotected-cell input"

Commit message: feat: support ordinary JLC fabrication and document complete materials
Parts:
- R56: value 1.82k/1% -> 1.69k/1%
Other:
- note added: "R40=2.21k: 403mA nominal; R55/TMR=69.8k, R56/ITERM=1.69k (all 1%). USB500 only after host configuration; suspend disables charging"
- note removed: "R40=2.21k: 403mA nominal; R55/TMR=69.8k, R56/ITERM=1.82k (all 1%). USB500 only after host configuration; suspend disables charging"
